File: 16550.sch (KiCad schematic (older format))
At the start: 7 parts, among them J16 DSUB-9, U13 PAL16L8, U14 74AHC1G04, U15 16550, U16 max235cpg

Commit message: adding changes
Parts:
- gave numbers to parts that had none: 2
Changed lines of the file:
@@
 $Descr A4 11693 8268
 encoding utf-8
-Sheet 3 3
+Sheet 3 4
 Title ""
 Date ""
@@
 Connection ~ 6150 1550
 $Comp
-L Device:C C?
+L Device:C C301
 U 1 1 60F65FED
 P 6150 1250
-F 0 "C?" H 6265 1296 50  0000 L CNN
+F 0 "C301" H 6265 1296 50  0000 L CNN
 F 1 "0.1uF" H 6265 1205 50  0000 L CNN
 F 2 "" H 6188 1100 50  0001 C CNN
@@
 $EndComp
 $Comp
-L power:GND #PWR?
+L power:GND #PWR0132
 U 1 1 60F66904
 P 6150 1100
-F 0 "#PWR?" H 6150 850 50  0001 C CNN
+F 0 "#PWR0132" H 6150 850 50  0001 C CNN
 F 1 "GND" H 6155 927 50  0000 C CNN
 F 2 "" H 6150 1100 50  0001 C CNN
@@
 $EndComp
 $Comp
-L power:VCC #PWR?
+L power:VCC #PWR0133
 U 1 1 60F6AFA9
 P 8050 1400
-F 0 "#PWR?" H 8050 1250 50  0001 C CNN
+F 0 "#PWR0133" H 8050 1250 50  0001 C CNN
 F 1 "VCC" V 8065 1528 50  0000 L CNN
 F 2 "" H 8050 1400 50  0001 C CNN
@@
 Connection ~ 8050 1400
 $Comp
-L Device:C C?
+L Device:C C302
 U 1 1 60F6AFB2
 P 8050 1100
-F 0 "C?" H 8165 1146 50  0000 L CNN
+F 0 "C302" H 8165 1146 50  0000 L CNN
 F 1 "0.1uF" H 8165 1055 50  0000 L CNN
 F 2 "" H 8088 950 50  0001 C CNN
@@
 $EndComp
 $Comp
-L power:GND #PWR?
+L power:GND #PWR0134
 U 1 1 60F6AFB8
 P 8050 950
-F 0 "#PWR?" H 8050 700 50  0001 C CNN
+F 0 "#PWR0134" H 8050 700 50  0001 C CNN
 F 1 "GND" H 8055 777 50  0000 C CNN
 F 2 "" H 8050 950 50  0001 C CNN

Commit message: tweaked a few things
Parts:
- removed C302: 0.1uF, symbol Device:C
Changed lines of the file:
@@
-	-1   0    0    1
-$EndComp
-$Comp
-L power:VCC #PWR0133
-U 1 1 60F6AFA9
-P 8050 1400
-F 0 "#PWR0133" H 8050 1250 50  0001 C CNN
-F 1 "VCC" V 8065 1528 50  0000 L CNN
-F 2 "" H 8050 1400 50  0001 C CNN
-F 3 "" H 8050 1400 50  0001 C CNN
-	1    8050 1400
-	0    1    1    0
-$EndComp
-Wire Wire Line
-	7800 1400 8050 1400
-Wire Wire Line
-	8050 1400 8050 1250
-Connection ~ 8050 1400
-$Comp
-L Device:C C302
-U 1 1 60F6AFB2
-P 8050 1100
-F 0 "C302" H 8165 1146 50  0000 L CNN
-F 1 "0.1uF" H 8165 1055 50  0000 L CNN
-F 2 "" H 8088 950 50  0001 C CNN
-F 3 "~" H 8050 1100 50  0001 C CNN
-	1    8050 1100
-	1    0    0    -1
-$EndComp
-$Comp
-L power:GND #PWR0134
-U 1 1 60F6AFB8
-P 8050 950
-F 0 "#PWR0134" H 8050 700 50  0001 C CNN
-F 1 "GND" H 8055 777 50  0000 C CNN
-F 2 "" H 8050 950 50  0001 C CNN
-F 3 "" H 8050 950 50  0001 C CNN
-	1    8050 950
 	-1   0    0    1
 $EndComp

Commit message: made final adjustments to all the designes
Parts:
- removed U14: 74AHC1G04, symbol 74xGxx:74AHC1G04
- C301: footprint (none) -> Capacitor_SMD:CP_Elec_3x5.3
- J301: renamed from J16; footprint DSUB-9 -> parts:DSUB-9
- U301: renamed from U13; footprint (none) -> Package_DIP:DIP-20_W7.62mm_SMDSocket_SmallPads
- U303: renamed from U16; footprint max235cpg -> parts:max235cpg
- renumbered U15 to U302
Connections:
- net GND: now also U302.14 (~CS2~)
Changed lines of the file:
@@
 $Descr A4 11693 8268
 encoding utf-8
-Sheet 3 6
+Sheet 3 8
 Title ""
 Date ""
@@
 $EndDescr
 $Comp
-L Interface_UART:16550 U15
+L Interface_UART:16550 U302
 U 1 1 60D0B4A1
 P 5900 3250
-F 0 "U15" H 5900 5131 50  0000 C CNN
+F 0 "U302" H 5900 5131 50  0000 C CNN
 F 1 "16550" H 5900 5040 50  0000 C CNN
 F 2 "Package_DIP:DIP-40_W15.24mm" H 5900 3250 50  0001 C CIN
@@
 P 2700 3550
 AR Path="/607EFB7A/60D2EA4E" Ref="U?"  Part="1"
-AR Path="/60D0ACC9/60D2EA4E" Ref="U13"  Part="1"
-F 0 "U13" H 2700 4431 50  0000 C CNN
+AR Path="/60D0ACC9/60D2EA4E" Ref="U301"  Part="1"
+F 0 "U301" H 2700 4431 50  0000 C CNN
 F 1 "PAL16L8" H 2700 4340 50  0000 C CNN
-F 2 "" H 2700 3550 50  0001 C CNN
+F 2 "Package_DIP:DIP-20_W7.62mm_SMDSocket_SmallPads" H 2700 3550 50  0001 C CNN
 F 3 "" H 2700 3550 50  0001 C CNN
 	1    2700 3550
@@
 P 2700 4150
 AR Path="/607EFB7A/60D2EA83" Ref="#PWR?"  Part="1"
-AR Path="/60D0ACC9/60D2EA83" Ref="#PWR06"  Part="1"
-F 0 "#PWR06" H 2700 3900 50  0001 C CNN
+AR Path="/60D0ACC9/60D2EA83" Ref="#PWR0302"  Part="1"
+F 0 "#PWR0302" H 2700 3900 50  0001 C CNN
 F 1 "GND" H 2705 3977 50  0000 C CNN
 F 2 "" H 2700 4150 50  0001 C CNN
@@
 P 2700 2850
 AR Path="/607EFB7A/60D2EA89" Ref="#PWR?"  Part="1"
-AR Path="/60D0ACC9/60D2EA89" Ref="#PWR02"  Part="1"
-F 0 "#PWR02" H 2700 2700 50  0001 C CNN
+AR Path="/60D0ACC9/60D2EA89" Ref="#PWR0301"  Part="1"
+F 0 "#PWR0301" H 2700 2700 50  0001 C CNN
 F 1 "VCC" V 2715 2977 50  0000 L CNN
 F 2 "" H 2700 2850 50  0001 C CNN
@@
 	4900 2950 4850 2950
 Wire Wire Line
-	3200 3050 4000 3050
-$Comp
-L 74xGxx:74AHC1G04 U14
-U 1 1 60D4C4C9
-P 4400 3250
-F 0 "U14" H 4375 3517 50  0000 C CNN
-F 1 "74AHC1G04" H 4375 3426 50  0000 C CNN
-F 2 "" H 4400 3250 50  0001 C CNN
-F 3 "http://www.ti.com/lit/sg/scyt129e/scyt129e.pdf" H 4400 3250 50  0001 C CNN
-	1    4400 3250
-	1    0    0    -1
-$EndComp
-Wire Wire Line
-	4000 3050 4000 3250
-Wire Wire Line
-	4000 3250 4100 3250
-Wire Wire Line
 	4600 3050 4600 3150
-Connection ~ 4000 3050
-Connection ~ 4600 3050
-Wire Wire Line
-	4000 3050 4600 3050
 Wire Wire Line
 	4600 3050 4900 3050
 Wire Wire Line
 	4600 3150 4900 3150
-Wire Wire Line
-	4650 3250 4900 3250
 Wire Wire Line
 	3200 3150 3350 3150
@@
 	4900 3450 4800 3450
 $Comp
-L max235cpg:max235cpg U16
+L max235cpg:max235cpg U303
 U 1 1 60D9FDB4
 P 8050 2050
-F 0 "U16" H 9350 2437 60  0000 C CNN
+F 0 "U303" H 9350 2437 60  0000 C CNN
 F 1 "max235cpg" H 9350 2331 60  0000 C CNN
-F 2 "max235cpg" H 9350 2290 60  0001 C CNN
+F 2 "parts:max235cpg" H 9350 2290 60  0001 C CNN
 F 3 "" H 8050 2050 60  0000 C CNN
 	1    8050 2050
@@
 $EndComp
 $Comp
-L DSUB-9:DSUB-9 J16
+L DSUB-9:DSUB-9 J301
 U 1 1 60DA5AC8
 P 9200 4050
-F 0 "J16" H 10028 3703 60  0000 L CNN
+F 0 "J301" H 10028 3703 60  0000 L CNN
 F 1 "DSUB-9" H 10028 3597 60  0000 L CNN
-F 2 "DSUB-9" H 9800 3690 60  0001 C CNN
+F 2 "parts:DSUB-9" H 9800 3690 60  0001 C CNN
 F 3 "" H 9200 4050 60  0000 C CNN
 	1    9200 4050
@@
 ~CTS
 $Comp
-L power:GND #PWR010
+L power:GND #PWR0307
 U 1 1 60DCED36
 P 8050 3050
-F 0 "#PWR010" H 8050 2800 50  0001 C CNN
+F 0 "#PWR0307" H 8050 2800 50  0001 C CNN
 F 1 "GND" V 8055 2922 50  0000 R CNN
 F 2 "" H 8050 3050 50  0001 C CNN
@@
 $EndComp
 $Comp
-L power:VCC #PWR011
+L power:VCC #PWR0308
 U 1 1 60DCF073
 P 8050 3150
-F 0 "#PWR011" H 8050 3000 50  0001 C CNN
+F 0 "#PWR0308" H 8050 3000 50  0001 C CNN
 F 1 "VCC" H 8065 3323 50  0000 C CNN
 F 2 "" H 8050 3150 50  0001 C CNN
@@
 	10850 2350 10850 2450
 $Comp
-L power:GND #PWR013
+L power:GND #PWR0310
 U 1 1 60E61994
 P 10850 2450
-F 0 "#PWR013" H 10850 2200 50  0001 C CNN
+F 0 "#PWR0310" H 10850 2200 50  0001 C CNN
 F 1 "GND" V 10855 2322 50  0000 R CNN
 F 2 "" H 10850 2450 50  0001 C CNN
@@
 DCDIN
 $Comp
-L power:GND #PWR012
+L power:GND #PWR0309
 U 1 1 60E7F24A
 P 8800 4450
-F 0 "#PWR012" H 8800 4200 50  0001 C CNN
+F 0 "#PWR0309" H 8800 4200 50  0001 C CNN
 F 1 "GND" V 8805 4322 50  0000 R CNN
 F 2 "" H 8800 4450 50  0001 C CNN
@@
 	4800 4250 4900 4250
 $Comp
-L power:GND #PWR07
+L power:GND #PWR0303
 U 1 1 60EA5E4F
 P 4450 4200
-F 0 "#PWR07" H 4450 3950 50  0001 C CNN
+F 0 "#PWR0303" H 4450 3950 50  0001 C CNN
 F 1 "GND" V 4455 4072 50  0000 R CNN
 F 2 "" H 4450 4200 50  0001 C CNN
@@
 	4750 4050 4900 4050
 $Comp
-L power:GND #PWR09
+L power:GND #PWR0304
 U 1 1 60EE692A
 P 5900 4950
-F 0 "#PWR09" H 5900 4700 50  0001 C CNN
+F 0 "#PWR0304" H 5900 4700 50  0001 C CNN
 F 1 "GND" H 5905 4777 50  0000 C CNN
 F 2 "" H 5900 4950 50  0001 C CNN
@@
 $EndComp
 $Comp
-L power:VCC #PWR08
+L power:VCC #PWR0306
 U 1 1 60EE6A9F
 P 6150 1550
-F 0 "#PWR08" H 6150 1400 50  0001 C CNN
+F 0 "#PWR0306" H 6150 1400 50  0001 C CNN
 F 1 "VCC" V 6165 1678 50  0000 L CNN
 F 2 "" H 6150 1550 50  0001 C CNN
@@
 F 0 "C301" H 6265 1296 50  0000 L CNN
 F 1 "0.1uF" H 6265 1205 50  0000 L CNN
-F 2 "" H 6188 1100 50  0001 C CNN
+F 2 "Capacitor_SMD:CP_Elec_3x5.3" H 6188 1100 50  0001 C CNN
 F 3 "~" H 6150 1250 50  0001 C CNN
 	1    6150 1250
@@
 $EndComp
 $Comp
-L power:GND #PWR0132
+L power:GND #PWR0305
 U 1 1 60F66904
 P 6150 1100
-F 0 "#PWR0132" H 6150 850 50  0001 C CNN
+F 0 "#PWR0305" H 6150 850 50  0001 C CNN
 F 1 "GND" H 6155 927 50  0000 C CNN
 F 2 "" H 6150 1100 50  0001 C CNN
@@
 $EndComp
 Wire Wire Line
+	3200 3050 4600 3050
+Connection ~ 4600 3050
+Wire Wire Line
+	4450 3250 4450 4200
+Wire Wire Line
+	4450 3250 4900 3250
+Connection ~ 4450 4200
+Wire Wire Line
 	3200 3250 3350 3250
