File: 7seg&led.sch (KiCad schematic (older format))
At the start: 27 parts, among them U401 PAL16L8, U402 74LS27, U403 74AHC373, U404 74LS27, U405 PAL16L8, U406 PAL16L8, U407 74LS27, U408 74AHC373, U409 74AHC373, U410 MAN71A, U411 MAN71A

Commit message: Updated 7seg&led wiring
The 8 LEDs power wasn't connected and the OE to ground.
Connections:
- wire segments 100 -> 104
Changed lines of the file:
@@
 $Descr A4 11693 8268
 encoding utf-8
-Sheet 4 6
+Sheet 1 1
 Title ""
 Date ""
@@
 L power:GND #PWR0147
 U 1 1 60AF626D
-P 3650 3650
-F 0 "#PWR0147" H 3650 3400 50  0001 C CNN
-F 1 "GND" H 3655 3477 50  0000 C CNN
-F 2 "" H 3650 3650 50  0001 C CNN
-F 3 "" H 3650 3650 50  0001 C CNN
-	1    3650 3650
-	1    0    0    -1
+P 3650 3900
+F 0 "#PWR0147" H 3650 3650 50  0001 C CNN
+F 1 "GND" H 3655 3727 50  0000 C CNN
+F 2 "" H 3650 3900 50  0001 C CNN
+F 3 "" H 3650 3900 50  0001 C CNN
+	1    3650 3900
+	1    0    0    -1
+$EndComp
+Wire Wire Line
+	3650 3650 3650 3850
+Wire Wire Line
+	3650 3850 3150 3850
+Wire Wire Line
+	3150 3850 3150 3350
+Connection ~ 3650 3850
+Wire Wire Line
+	3650 3850 3650 3900
+$Comp
+L power:+5V #PWR?
+U 1 1 60954095
+P 3650 2050
+F 0 "#PWR?" H 3650 1900 50  0001 C CNN
+F 1 "+5V" V 3665 2178 50  0000 L CNN
+F 2 "" H 3650 2050 50  0001 C CNN
+F 3 "" H 3650 2050 50  0001 C CNN
+	1    3650 2050
+	0    1    1    0
 $EndComp
 $EndSCHEMATC

Commit message: tweaked a few things
Changed lines of the file:
@@
 $Descr A4 11693 8268
 encoding utf-8
-Sheet 1 1
+Sheet 4 6
 Title ""
 Date ""
@@
 	5550 2900 5550 2750
 Connection ~ 5550 2750
-Wire Wire Line
-	5350 3200 5550 3200
 Wire Wire Line
 	5550 3200 5550 2900
@@
 	3650 3850 3650 3900
 $Comp
-L power:+5V #PWR?
+L power:+5V #PWR0148
 U 1 1 60954095
 P 3650 2050
-F 0 "#PWR?" H 3650 1900 50  0001 C CNN
+F 0 "#PWR0148" H 3650 1900 50  0001 C CNN
 F 1 "+5V" V 3665 2178 50  0000 L CNN
 F 2 "" H 3650 2050 50  0001 C CNN
@@
 	0    1    1    0
 $EndComp
+Wire Wire Line
+	5300 3200 5550 3200
 $EndSCHEMATC

Commit message: made some modifications
Parts:
- removed U402, U404, U407: 74LS27, symbol 74xx:74LS27
- added U? (x6): 74AHC1G08, symbol 74xGxx:74AHC1G08
Connections:
- net labels added: A0
- wire segments 104 -> 118

Commit message: made final adjustments to all the designes
Parts:
- removed U? (x6): 74AHC1G08, symbol 74xGxx:74AHC1G08
- added U401, U404: 74LS21, Package_DIP:DIP-14_W7.62mm_SMDSocket_SmallPads, symbol 74xx:74LS21
- D401, D402, D403, D404, D405, D406, D407, D408: footprint (none) -> LED_SMD:LED_1812_4532Metric
- R401, R402, R403, R404, R405, R406, R407, R408: footprint (none) -> Resistor_SMD:R_0402_1005Metric
- U402: renamed from U401; footprint (none) -> Package_DIP:DIP-20_W7.62mm_SMDSocket_SmallPads
- U403, U405, U406: footprint (none) -> Package_DIP:DIP-20_W7.62mm_SMDSocket_SmallPads
- U407: renamed from U408; footprint (none) -> Package_DIP:DIP-20_W7.62mm_SMDSocket_SmallPads
- U408: renamed from U409; footprint (none) -> Package_DIP:DIP-20_W7.62mm_SMDSocket_SmallPads
- renumbered U410 to U409, U411 to U410
Connections:
- net A16: now also U401.1, U404.1, U404.9
- net A17: now also U401.2, U404.10, U404.2
- net A18: now also U401.4, U404.12, U404.4
- net A19: now also U401.5, U404.13, U404.5
- net GND: now also U401.7 (GND), U404.7 (GND)
- net VCC: now also U401.14 (VCC), U404.14 (VCC)
- net at U405.18 (IO2): now also U404.6
- net at U406.18 (IO2): now also U404.8
- net at U402.18 (IO2): now also U401.6
Other:
- moved on the sheet: D401, D402, D403, D404, D405, D406, D407, D408, R401, R402, R403, R404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
