File: 8259.sch (KiCad schematic (older format))
At the start: 10 parts

Commit message: made final adjustments to all the designes
Parts:
- removed U?: 74LS00, symbol 74xx:74LS00
- removed U?: 4001, symbol 4xxx:4001
- added C701: 0.1uF, Capacitor_SMD:CP_Elec_3x5.3, symbol Device:C
- added U701: 74LS11, Package_DIP:DIP-14_W7.62mm_SMDSocket_SmallPads, symbol 74xx:74LS11
- added unit 2 of U704
- added unit 5 of U704
- J701: renamed from J?; footprint (none) -> Connector_JST:JST_GH_BM04B-GHS-TBT_1x04-1MP_P1.25mm_Vertical
- R701, R702, R703: renamed from R?; footprint (none) -> Resistor_SMD:R_0402_1005Metric
- SW701: renamed from SW?; footprint (none) -> Button_Switch_SMD:SW_SPST_B3U-1000P
- U703: renamed from U?; footprint (none) -> Package_DIP:DIP-20_W7.62mm_SMDSocket_SmallPads
- U704: renamed from U?; footprint (none) -> Package_DIP:DIP-14_W7.62mm_SMDSocket_SmallPads
- gave numbers to parts that had none: 1
Connections:
- net labels added: INTR, IR1, IR2, IR3, VCC, ~INTA, ~RD, ~WR
- net labels removed: 16550INTR, 8254, INT, INTA, IRQ, RD, WR
Other:
- moved on the sheet: J701, R701, R702, R703, SW701, U702, U703, U704A
