File: proj5.kicad_pcb (KiCad board)
At the start: 2 copper layers, 134 parts, among them J101 Screw_Terminal_01x02, J102 Conn_01x08_Male, J103 Conn_01x08_Male, J104 Conn_01x12_Male, J105 Conn_01x04_Male, J106 Conn_01x08_Male, J107 Conn_01x08_Male, J201 Conn_01x08_Male, J202 Conn_01x08_Male, J203 Conn_01x08_Male, J204 Conn_01x08_Male, J205 Conn_01x08_Male, J206 Conn_01x08_Male, J207 Conn_01x08_Male, J208 Conn_01x08_Male, J209 Conn_01x08_Male, J301 DSUB-9, J501 Conn_01x03_Male, J502 Conn_01x02_Male, J503 Conn_01x03_Male, J701 Conn_01x04_Male, SW101 SW_Push, SW102 SW_Push, SW701 SW_Push, SW801 SW_Push, SW802 SW_Push, SW803 SW_Push, SW804 SW_Push, SW805 SW_Push, SW806 SW_Push, SW807 SW_Push, SW808 SW_Push, SW809 SW_Push, SW810 SW_Push, SW811 SW_Push, SW812 SW_Push, SW813 SW_Push, SW814 SW_Push, SW815 SW_Push, SW816 SW_Push, SW817 SW_Push, SW818 SW_Push, SW819 SW_Push, SW820 SW_Push, SW821 SW_Push, SW822 SW_Push, U101 74LS245, U102 74LS245, U103 8284, U104 8086_Min_Mode, U105 74LS373, U106 74AHC373, U107 74AHC373, U201 74LS21, U202 PAL16L8, U203 8255, U204 8255, U205 8255, U301 PAL16L8, U302 16550, U303 max235cpg, U401 74LS21, U402 PAL16L8, U403 74AHC373, U404 74LS21, U405 PAL16L8, U406 PAL16L8, U407 74AHC373, U408 74AHC373, U409 MAN71A, U410 MAN71A, U501 74LS08, U502 PAL16L8, U503 8254, U504 PAL16L8, U601 28F010, U602 28F010, U603 74LS04, U604 PAL16L8, U605 CY7C199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

Commit message: adjusted and incorperated 8dipswitch to pcb
Parts:
- added R901: R_US, Resistor_SMD:R_0805_2012Metric, F.Cu at (55.9, 120.7)
- added R902: R_US, Resistor_SMD:R_0805_2012Metric, F.Cu at (60.0, 120.7)
- added R903: R_US, Resistor_SMD:R_0805_2012Metric, F.Cu at (68.6, 135.9)
- added R904: R_US, Resistor_SMD:R_0805_2012Metric, F.Cu at (64.8, 120.7)
- added R905: R_US, Resistor_SMD:R_0805_2012Metric, F.Cu at (69.8, 120.7)
- added R906: R_US, Resistor_SMD:R_0805_2012Metric, F.Cu at (67.3, 141.0)
- added R907: R_US, Resistor_SMD:R_0805_2012Metric, F.Cu at (74.9, 120.7)
- added R908: R_US, Resistor_SMD:R_0805_2012Metric, F.Cu at (67.3, 146.1)
- added SW901: SW_DIP_x08, Button_Switch_SMD:SW_DIP_SPSTx08_Slide_6.7x21.88mm_W6.73mm_P2.54mm_LowProfile_JPin, F.Cu at (57.1, 135.9)
- added U901: PAL16L8, Package_DIP:DIP-20_W7.62mm_SMDSocket_SmallPads, F.Cu at (57.1, 101.6)
- added U902: 74LS244, Package_DIP:DIP-20_W7.62mm_SMDSocket_SmallPads, F.Cu at (106.7, 120.7)
- moved U802 175.8 mm to (133.0, 192.0)
- moved SW801 80.5 mm to (141.0, 138.0)
- moved C801 64.5 mm to (125.0, 135.0)
- moved SW802 59.6 mm to (133.0, 133.3)
- moved U404 57.4 mm to (119.0, 37.0)
- moved J501 54.7 mm to (68.0, 28.0)
- moved J502 54.7 mm to (68.0, 15.0)
- moved J503 54.7 mm to (68.0, 0.00)
- moved SW813 46.9 mm to (86.0, 182.0), turned to 90 degrees
- moved SW804 45.0 mm to (68.0, 173.0)
- moved SW810 41.6 mm to (77.0, 190.0)
- moved D404 40.8 mm to (230.0, 120.0), turned to 180 degrees
- moved U502 40.7 mm to (144.0, 82.0)
- moved SW805 36.5 mm to (68.0, 182.0)
- moved C501 35.2 mm to (96.0, -9.00), turned to 180 degrees
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Connections:
- net Net-(U201-Pad6) renamed /8255/4dec
- net Net-(U801-Pad12) renamed A17,18,19
Routing:
- net GND: track 52.2 -> 1016.4 mm, vias 0 -> 22
- net +5V: track 34.1 -> 944.3 mm, vias 2 -> 42
- net D5: track 95.0 -> 728.8 mm, vias 4 -> 19
- net D1: track 103.2 -> 720.0 mm, vias 0 -> 7
- net D7: track 95.2 -> 701.7 mm, vias 4 -> 18
- net D6: track 95.4 -> 684.1 mm, vias 4 -> 17
- net D2: track 102.6 -> 676.3 mm, vias 0 -> 7
- net D4: track 95.0 -> 661.0 mm, vias 4 -> 18
- net A17: track 28.6 -> 577.7 mm, vias 0 -> 27
- net A18: track 0.00 -> 489.3 mm, vias 0 -> 8
- net A19: track 0.00 -> 453.7 mm, vias 0 -> 12
- net A5: track 206.0 -> 647.8 mm, vias 8 -> 20
- net A16: track 28.6 -> 469.9 mm, vias 0 -> 16
- net IR1: track 0.00 -> 433.4 mm
- net ~RD: track 171.7 -> 584.9 mm, vias 4 -> 8
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- added copper zone on PWR, net +5V
- added copper zone on GND, net GND
Other:
- copper layers 2 -> 4

Commit message: finished pcb layout
Parts:
- J101: footprint TerminalBlock_4Ucon:TerminalBlock_4Ucon_1x02_P3.50mm_Horizontal -> TerminalBlock_Phoenix:TerminalBlock_Phoenix_MKDS-1,5-2-5.08_1x02_P5.08mm_Horizontal
- moved R905 15.3 mm to (85.1, 119.4)
- moved R907 15.3 mm to (90.2, 119.4)
- moved D101 10.4 mm to (310.4, 38.1)
- moved C103 9.57 mm to (315.0, 7.62)
- moved C301 7.14 mm to (279.2, 188.0)
- moved R904 6.84 mm to (71.1, 118.1)
- moved R903 6.84 mm to (74.9, 133.3)
- moved R908 6.84 mm to (73.7, 143.5)
- moved SW901 6.84 mm to (63.5, 133.3)
- moved U901 6.84 mm to (63.5, 99.1)
- moved R901 6.84 mm to (62.2, 118.1)
- moved R902 6.84 mm to (66.4, 118.1)
- moved R906 6.84 mm to (73.7, 138.4)
- moved J101 4.54 mm to (353.1, -20.3)
Routing:
- net GND: track 1016.4 -> 64.0 mm, vias 22 -> 76
- net +5V: track 944.3 -> 58.3 mm, vias 42 -> 72
- net ~WR: track 410.6 -> 1081.4 mm, vias 17 -> 24
- net RESET: track 61.8 -> 590.3 mm, vias 2 -> 8
- net D0: track 510.4 -> 1020.2 mm, vias 4 -> 8
- net A1: track 458.5 -> 964.4 mm, vias 21 -> 30
- net D3: track 471.7 -> 976.3 mm, vias 10 -> 19
- net PCLK: track 0.00 -> 459.1 mm, vias 0 -> 4
- net ~RD: track 584.9 -> 1014.3 mm, vias 8 -> 18
- net A2: track 550.1 -> 951.7 mm, vias 12 -> 19
- net D5: track 728.8 -> 1128.0 mm, vias 19 -> 27
- net IR2: track 0.00 -> 384.2 mm
- net D2: track 676.3 -> 1035.3 mm, vias 7 -> 11
- net D4: track 661.0 -> 1000.0 mm, vias 18 -> 23
- net D6: track 684.1 -> 1001.0 mm, vias 17 -> 24
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Other:
- board outline added: 312.9 x 241.8 mm
